Commit message: パラメータ変更

File: urdf/base/base.urdf.xacro (robot description, xacro)
@@ -16,14 +16,13 @@
       </visual>
       <collision>
-        <origin xyz="0.0 0.0 0.0" rpy="${M_PI/2} 0 ${M_PI/2}"/>
+        <origin xyz="0.0 0.0 0.27" rpy="0 0 0"/>
         <geometry>
-          <mesh filename="package://infant3/meshes/STL/base.stl" scale="0.001 0.001 0.001"/>
+          <box size="0.700 0.500 0.535"/>
         </geometry>
       </collision>
       <inertial>
         <origin xyz="0.0 0.0 0.0" rpy="${M_PI/2} 0 ${M_PI/2}"/>
-        <box_inertial mass="5.0" height="0.5" width="0.5" depth="0.5"/>
-        <mass value="43.24"/>
-        <inertia ixx="4.115" ixy="0" ixz="0" iyz="0" iyy="4.207" izz="4.076"/>
+        <mass value="26"/>
+        <inertia ixx="4.941" ixy="0" ixz="0" iyz="0" iyy="5.327" izz="0.849"/>
       </inertial>
     </link>

File: urdf/caster/caster.urdf.xacro (robot description, xacro)
@@ -13,4 +13,5 @@
         <geometry>
           <mesh filename="package://infant3/meshes/STL/caster.stl" scale="0.001 0.001 0.001"/>
+          <sphere radius="0.050"/>
         </geometry>
       </visual>
@@ -18,5 +19,6 @@
         <origin xyz="0 0.0125 0" rpy="${M_PI/2} 0 ${-M_PI/2}"/>
         <geometry>
-          <mesh filename="package://infant3/meshes/STL/caster.stl" scale="0.001 0.001 0.001"/>
+          <!--mesh filename="package://infant3/meshes/STL/caster.stl" scale="0.001 0.001 0.001"/-->
+          <sphere radius="0.050"/>
         </geometry>
       </collision>
