Commit message: updating urdf and stl

File: robot/cats.urdf (robot description, URDF)
Before this commit: robot cats, 1 links, 0 joints
Links:
- removed link base_footprint
- added link base_link

File: urdf/wheel/wheel.urdf.xacro (robot description, xacro)
@@ -2,5 +2,5 @@
 <robot xmlns:xacro="http://ros.org/wiki/xacro">
   <xacro:include filename="$(find cats)/urdf/common.xacro"/>
-  <property name="wheel_radius" value="0.125"/>
+  <property name="wheel_radius" value="0.1245"/>
   <property name="wheel_width" value="0.073"/>
   <property name="wheel_mass" value="4.0"/>
@@ -11,9 +11,9 @@
       <child link="${prefix}_wheel_link"/>
       <insert_block name="joint_axis"/>
-      <limit velocity="30" effort="23"/>
+      <limit velocity="11.64" effort="11.25"/>
     </joint>
     <link name="${prefix}_wheel_link">
       <visual>
-        <origin xyz="-0.0365 0 0" rpy="0 0 0"/>
+        <origin xyz="0 0 0" rpy="0 0 0"/>
         <geometry>
           <mesh filename="package://cats/meshes/STL/wheel.stl" scale="0.001 0.001 0.001"/>
@@ -21,5 +21,5 @@
       </visual>
       <collision>
-        <origin xyz="-0.0365 0 0" rpy="0 0 0"/>
+        <origin xyz="0 0 0" rpy="0 0 0"/>
         <geometry>
           <mesh filename="package://cats/meshes/STL/wheel.stl" scale="0.001 0.001 0.001"/>
@@ -27,5 +27,5 @@
       </collision>
       <inertial>
-        <origin xyz="-0.0365 0 0" rpy="0 0 0"/>
+        <origin xyz="0 0 0" rpy="0 0 0"/>
         <cylinder_inertial mass="${wheel_mass}"
           radius="${wheel_radius}" length="${wheel_width}"/>

Commit message: add robot_state.launch

File: robot/cats.urdf (robot description, URDF)
Before this commit: robot cats, 1 links, 0 joints
Links:
- added link camera_link
Joints:
- added joint body_link2realsense: type fixed, parent body_link, child camera_link, origin xyz=0.04 0 0.75 rpy=0 0.7853981633974483 0
