Commit message: 修正

File: urdf/sensors/camera.urdf.xacro (robot description, xacro)
@@ -4,5 +4,8 @@
   <xacro:macro name="camera" params="prefix parent *joint_origin">
     <joint name="${prefix}_camera_joint" type="fixed">
+      <xacro:insert_block name="joint_origin"/>
+      <!--
       <axis xyz="0 1 0" />
+      -->
       <parent link="${parent}"/>
       <child link="${prefix}_camera"/>
@@ -12,5 +15,5 @@
         <origin xyz="0 0 0" rpy="0 0 0"/>
         <geometry>
-          <mesh filename="package://infant3/meshes/STL/camera.stl"/>
+          <mesh filename="package://infant3/meshes/STL/camera.stl" scale="0.001 0.001 0.001"/>
         </geometry>
       </visual>
@@ -18,5 +21,5 @@
         <origin xyz="0 0 0" rpy="0 0 0"/>
         <geometry>
-          <mesh filename="package://infant3/meshes/STL/camera.stl"/>
+          <mesh filename="package://infant3/meshes/STL/camera.stl" scale="0.001 0.001 0.001"/>
         </geometry>
       </collision>
@@ -28,9 +31,10 @@
     </link>
   </xacro:macro>
-  <xacro:macro name="camera_gazebo" params="prefix width height">
+  <xacro:macro name="camera_gazebo" params="prefix">
     <gazebo reference="${prefix}_camera">
       <sensor type="camera" name="${prefix}_camera_sensor">
-        <update_rate>30.0</update_rate>
-        <camera>
+        <!--visualize>false</visualize-->
+        <update_rate>30</update_rate>
+        <camera name="head">
           <horizontal_fov>1.3439035</horizontal_fov>
           <image>
@@ -43,5 +47,4 @@
             <far>300</far>
           </clip>
-          <!--
           <noise>
             <type>gaussian</type>
@@ -49,12 +52,11 @@
             <stddev>0.007</stddev>
           </noise>
-          -->
         </camera>
         <plugin name="gazebo_ros_${prefix}_camera_controller" filename="libgazebo_ros_camera.so">
           <alwaysOn>true</alwaysOn>
-          <updateRate>0.0</updateRate>
+          <updateRate>30.0</updateRate>
           <cameraName>${prefix}_camera</cameraName>
           <imageTopicName>/${prefix}_camera/image_raw</imageTopicName>
-          <cameraInfoTopicName>${prefix}_camera_info</cameraInfoTopicName>
+          <cameraInfoTopicName>/${prefix}_camera_info</cameraInfoTopicName>
           <frameName>${prefix}_camera</frameName>
           <hackBaseline>0.07</hackBaseline>

Commit message: cameraをwebcameraにリネーム

File: urdf/sensors/camera.urdf.xacro (robot description, xacro)
@@ -2,10 +2,8 @@
 <robot xmlns:xacro="http://ros.org/wiki/xacro">
   <xacro:include filename="$(find infant3)/urdf/common.xacro"/>
-  <xacro:macro name="camera" params="prefix parent *joint_origin">
+  <xacro:macro name="webcamera" params="prefix parent *joint_origin">
     <joint name="${prefix}_camera_joint" type="fixed">
       <xacro:insert_block name="joint_origin"/>
-      <!--
       <axis xyz="0 1 0" />
-      -->
       <parent link="${parent}"/>
       <child link="${prefix}_camera"/>
@@ -34,6 +32,5 @@
     <gazebo reference="${prefix}_camera">
       <sensor type="camera" name="${prefix}_camera_sensor">
-        <!--visualize>false</visualize-->
-        <update_rate>30</update_rate>
+        <update_rate>30.0</update_rate>
         <camera name="head">
           <horizontal_fov>1.3439035</horizontal_fov>
@@ -55,5 +52,5 @@
         <plugin name="gazebo_ros_${prefix}_camera_controller" filename="libgazebo_ros_camera.so">
           <alwaysOn>true</alwaysOn>
-          <updateRate>30.0</updateRate>
+          <updateRate>0.0</updateRate>
           <cameraName>${prefix}_camera</cameraName>
           <imageTopicName>/${prefix}_camera/image_raw</imageTopicName>
@@ -68,4 +65,6 @@
         </plugin>
       </sensor>
+      <mu1>0.2</mu1>
+      <mu2>0.2</mu2>
     </gazebo>
   </xacro:macro>

Commit message: カメラ姿勢を修正

File: urdf/sensors/camera.urdf.xacro (robot description, xacro)
@@ -5,5 +5,5 @@
     <joint name="${prefix}_camera_joint" type="fixed">
       <xacro:insert_block name="joint_origin"/>
-      <axis xyz="0 1 0" />
+      <axis xyz="0 0 1" />
       <parent link="${parent}"/>
       <child link="${prefix}_camera"/>
@@ -11,5 +11,5 @@
     <link name="${prefix}_camera">
       <visual>
-        <origin xyz="0 0 0" rpy="0 0 0"/>
+        <origin xyz="0 0 0" rpy="${M_PI/2} 0 ${M_PI/2}"/>
         <geometry>
           <mesh filename="package://infant3/meshes/STL/camera.stl" scale="0.001 0.001 0.001"/>

Commit message: update camera frame

File: urdf/sensors/camera.urdf.xacro (robot description, xacro)
@@ -28,4 +28,10 @@
       </inertial>
     </link>
+    <joint name="${prefix}_camera_optical_frame_joint" type="fixed">
+      <origin xyz="0.0 0.0 0.0" rpy="-1.57 0.0 -1.57"/>
+      <parent link="${prefix}_camera"/>
+      <child link="${prefix}_camera/optical_frame"/>
+    </joint>
+    <link name="${prefix}_camera/optical_frame"/>
   </xacro:macro>
   <xacro:macro name="camera_gazebo" params="prefix">
@@ -56,5 +62,5 @@
           <imageTopicName>/${prefix}_camera/image_raw</imageTopicName>
           <cameraInfoTopicName>/${prefix}_camera_info</cameraInfoTopicName>
-          <frameName>${prefix}_camera</frameName>
+          <frameName>${prefix}_camera/optical_frame</frameName>
           <hackBaseline>0.07</hackBaseline>
           <distortionK1>0.0</distortionK1>
