Commit message: update caster and body

File: urdf/body/body.urdf.xacro (robot description, xacro)
@@ -16,11 +16,11 @@
       </visual>
       <collision>
-        <origin xyz="0.0 0.0 0.2675" rpy="0 0 0"/>
+        <origin xyz="-0.240 0 0.04025" rpy="0 0 0"/>
         <geometry>
-          <box size="0.700 0.500 0.535"/>
+          <box size="0.525 0.400 0.2755"/>
         </geometry>
       </collision>
       <inertial>
-        <origin xyz="0.0 0.0 0.2675" rpy="0 0 0"/>
+        <origin xyz="-0.240 0 0" rpy="0 0 0"/>
         <mass value="26"/>
         <inertia ixx="4.941" ixy="0" ixz="0" iyz="0" iyy="5.327" izz="0.849"/>

File: urdf/caster/caster.urdf.xacro (robot description, xacro)
@@ -6,34 +6,91 @@
       <insert_block name="joint_origin"/>
       <parent link="${parent}"/>
-      <child link="${prefix}_caster_link"/>
+      <child link="${prefix}_caster_base_link"/>
     </joint>
-    <link name="${prefix}_caster_link">
+    <link name="${prefix}_caster_base_link">
       <visual>
-        <origin xyz="0 0.0125 0" rpy="${M_PI/2} 0 ${-M_PI/2}"/>
+        <origin xyz="0 0.144608 -0.214894" rpy="${M_PI/2} 0 ${-M_PI/2}"/>
         <geometry>
-          <mesh filename="package://cats/meshes/STL/caster.stl" scale="0.001 0.001 0.001"/>
-          <sphere radius="0.050"/>
+          <mesh filename="package://cats/meshes/STL/caster/caster_base.stl" scale="0.001 0.001 0.001"/>
         </geometry>
       </visual>
       <collision>
-        <origin xyz="0 0.0125 0" rpy="${M_PI/2} 0 ${-M_PI/2}"/>
+        <origin xyz="0 0 0" rpy="0 0 0"/>
         <geometry>
-          <!--mesh filename="package://cats/meshes/STL/caster.stl" scale="0.001 0.001 0.001"/-->
-          <sphere radius="0.050"/>
+          <cylinder radius="0.0365" length="0.023"/>
         </geometry>
       </collision>
       <inertial>
-        <origin xyz="0 0.0125 0" rpy="${M_PI/2} 0 ${-M_PI/2}"/>
-        <cylinder_inertial mass="0.550"
-          radius="0.050" length="0.025"/>
+        <origin xyz="0 0 0" rpy="0 0 0"/>
+        <cylinder_inertial mass="0.500" radius="0.0365" length="0.023"/>
+      </inertial>
+    </link>
+    <joint name="${prefix}_caster_arm_joint" type="continuous">
+      <origin xyz="0 0 -0.009" rpy="0 0 0"/>
+      <parent link="${prefix}_caster_base_link"/>
+      <child link="${prefix}_caster_arm_link"/>
+      <axis xyz="0 0 1"/>
+      <limit velocity="17.45" effort="7.5"/>
+    </joint>
+    <link name="${prefix}_caster_arm_link">
+      <visual>
+        <origin xyz="-0.144608 0 -0.205602" rpy="${M_PI/2} 0 0"/>
+        <geometry>
+          <mesh filename="package://cats/meshes/STL/caster/caster_arm.stl" scale="0.001 0.001 0.001"/>
+        </geometry>
+      </visual>
+      <collision>
+        <origin xyz="0 0 0" rpy="0 0 0"/>
+        <geometry>
+          <cylinder radius="0.0365" length="0.023"/>
+        </geometry>
+      </collision>
+      <inertial>
+        <origin xyz="0 0 0" rpy="0 0 0"/>
+        <cylinder_inertial mass="0.500" radius="0.0365" length="0.023"/>
+      </inertial>
+    </link>
+    <joint name="${prefix}_caster_wheel_joint" type="continuous">
+      <origin xyz="-0.044987 0 -0.101525" rpy="0 0 0"/>
+      <parent link="${prefix}_caster_arm_link"/>
+      <child link="${prefix}_caster_wheel_link"/>
+      <axis xyz="0 1 0"/>
+      <limit velocity="17.45" effort="7.5"/>
+    </joint>
+    <link name="${prefix}_caster_wheel_link">
+      <visual>
+        <origin xyz="-0.099621 0 -0.104369" rpy="${M_PI/2} 0 0"/>
+        <geometry>
+          <mesh filename="package://cats/meshes/STL/caster/caster_wheel.stl" scale="0.001 0.001 0.001"/>
+        </geometry>
+      </visual>
+      <collision>
+        <origin xyz="0 0 0" rpy="${M_PI/2} 0 0"/>
+        <geometry>
+          <cylinder radius="0.050" length="0.030"/>
+        </geometry>
+      </collision>
+      <inertial>
+        <origin xyz="0 0 0" rpy="${M_PI/2} 0 0"/>
+        <cylinder_inertial mass="0.500" radius="0.050" length="0.030"/>
       </inertial>
     </link>
   </xacro:macro>
   <xacro:macro name="caster_gazebo" params="prefix">
-    <gazebo reference="${prefix}_caster_link">
+    <gazebo reference="${prefix}_caster_base_link">
       <selfCollide>false</selfCollide>
       <mu1 value="0"/>
       <mu2 value="0"/>
     </gazebo>
+    <gazebo reference="${prefix}_caster_arm_link">
+      <selfCollide>false</selfCollide>
+      <mu1 value="0.05"/>
+      <mu2 value="0.05"/>
+    </gazebo>
+    <gazebo reference="${prefix}_caster_wheel_link">
+      <selfCollide>false</selfCollide>
+      <mu1 value="0.8"/>
+      <mu2 value="0.8"/>
+    </gazebo>
   </xacro:macro>
   </robot>

Commit message: add upper body

File: urdf/body/body.urdf.xacro (robot description, xacro)
@@ -27,4 +27,50 @@
       </inertial>
     </link>
+    <joint name="upper_body_joint" type="fixed">
+      <parent link="body_link"/>
+      <child link="upper_body_link"/>
+      <origin xyz="-0.214 0 ${0.3255-0.245/2+0.020}" rpy="0 0 0"/>
+    </joint>
+    <link name="upper_body_link">
+      <visual>
+        <origin xyz="0 0 0.25" rpy="0 0 0"/>
+        <geometry>
+          <box size="0.4 0.3 0.5"/>
+        </geometry>
+      </visual>
+      <collision>
+        <origin xyz="0 0 0.25" rpy="0 0 0"/>
+        <geometry>
+          <box size="0.4 0.3 0.5"/>
+        </geometry>
+      </collision>
+      <inertial>
+        <origin xyz="0 0 0.25" rpy="0 0 0"/>
+        <box_inertial mass="15" depth="0.4" height="0.5" width="0.3"/>
+      </inertial>
+    </link>
+    <joint name="pillar_joint" type="fixed">
+      <parent link="upper_body_link"/>
+      <child link="pillar_link"/>
+      <origin xyz="0.01 0 0.5" rpy="0 0 0"/>
+    </joint>
+    <link name="pillar_link">
+      <visual>
+        <origin xyz="0 0 ${0.255/2}" rpy="0 0 0"/>
+        <geometry>
+          <box size="0.140 0.100 0.255"/>
+        </geometry>
+      </visual>
+      <collision>
+        <origin xyz="0 0 ${0.255/2}" rpy="0 0 0"/>
+        <geometry>
+          <box size="0.140 0.100 0.255"/>
+        </geometry>
+      </collision>
+      <inertial>
+        <origin xyz="0 0 ${0.255/2}" rpy="0 0 0"/>
+        <box_inertial mass="1" depth="0.140" height="0.255" width="0.100"/>
+      </inertial>
+    </link>
   </xacro:macro>
   <xacro:macro name="body_gazebo">
@@ -34,4 +80,14 @@
       <mu2 value="0.05"/>
     </gazebo>
+    <gazebo reference="upper_body_link">
+      <selfCollide>false</selfCollide>
+      <mu1 value="0.05"/>
+      <mu2 value="0.05"/>
+    </gazebo>
+    <gazebo reference="pillar_link">
+      <selfCollide>false</selfCollide>
+      <mu1 value="0.05"/>
+      <mu2 value="0.05"/>
+    </gazebo>
   </xacro:macro>
 </robot>

Commit message: update xacro files

File: urdf/body/body.urdf.xacro (robot description, xacro)
@@ -4,5 +4,5 @@
   <xacro:macro name="body" params="parent *joint_origin">
     <joint name="body_link_joint" type="fixed">
-      <insert_block name="joint_origin"/>
+      <xacro:insert_block name="joint_origin"/>
       <parent link="${parent}"/>
       <child link="body_link"/>

File: urdf/caster/caster.urdf.xacro (robot description, xacro)
@@ -4,5 +4,5 @@
   <xacro:macro name="caster" params="prefix parent *joint_origin">
     <joint name="${prefix}_caster_joint" type="fixed">
-      <insert_block name="joint_origin"/>
+      <xacro:insert_block name="joint_origin"/>
       <parent link="${parent}"/>
       <child link="${prefix}_caster_base_link"/>

File: urdf/common.xacro (robot description, xacro)
@@ -1,5 +1,5 @@
 <?xml version="1.0"?>
 <robot xmlns:xacro="http://ros.org/wiki/xacro">
-  <property name="M_PI" value="3.14159274"/>
+  <xacro:property name="M_PI" value="3.14159274"/>
   <xacro:macro name="cylinder_inertial" params="mass radius length">
     <mass value="${mass}"/>

File: urdf/wheel/wheel.urdf.xacro (robot description, xacro)
@@ -2,13 +2,13 @@
 <robot xmlns:xacro="http://ros.org/wiki/xacro">
   <xacro:include filename="$(find cats)/urdf/common.xacro"/>
-  <property name="wheel_radius" value="0.1245"/>
-  <property name="wheel_width" value="0.073"/>
-  <property name="wheel_mass" value="4.0"/>
+  <xacro:property name="wheel_radius" value="0.1245"/>
+  <xacro:property name="wheel_width" value="0.073"/>
+  <xacro:property name="wheel_mass" value="4.0"/>
   <xacro:macro name="wheel" params="prefix parent *joint_origin *joint_axis">
     <joint name="${prefix}_wheel_joint" type="continuous">
-      <insert_block name="joint_origin"/>
+      <xacro:insert_block name="joint_origin"/>
       <parent link="${parent}"/>
       <child link="${prefix}_wheel_link"/>
-      <insert_block name="joint_axis"/>
+      <xacro:insert_block name="joint_axis"/>
       <limit velocity="11.64" effort="11.25"/>
     </joint>

Commit message: update color

File: urdf/body/body.urdf.xacro (robot description, xacro)
@@ -14,4 +14,7 @@
           <mesh filename="package://cats/meshes/STL/body.stl" scale="0.001 0.001 0.001"/>
         </geometry>
+        <material name="gray">
+          <color rgba="0.8 0.8 0.8 1.0"/>
+        </material>
       </visual>
       <collision>
@@ -38,4 +41,6 @@
           <box size="0.4 0.3 0.5"/>
         </geometry>
+        <material name="gray">
+        </material>
       </visual>
       <collision>
@@ -61,4 +66,6 @@
           <box size="0.140 0.100 0.255"/>
         </geometry>
+        <material name="gray">
+        </material>
       </visual>
       <collision>
@@ -79,4 +86,5 @@
       <mu1 value="0.05"/>
       <mu2 value="0.05"/>
+      <material>Gazebo/Gray</material>
     </gazebo>
     <gazebo reference="upper_body_link">
@@ -84,4 +92,5 @@
       <mu1 value="0.05"/>
       <mu2 value="0.05"/>
+      <material>Gazebo/Gray</material>
     </gazebo>
     <gazebo reference="pillar_link">
@@ -89,4 +98,5 @@
       <mu1 value="0.05"/>
       <mu2 value="0.05"/>
+      <material>Gazebo/Gray</material>
     </gazebo>
   </xacro:macro>

File: urdf/caster/caster.urdf.xacro (robot description, xacro)
@@ -14,4 +14,6 @@
           <mesh filename="package://cats/meshes/STL/caster/caster_base.stl" scale="0.001 0.001 0.001"/>
         </geometry>
+        <material name="gray">
+        </material>
       </visual>
       <collision>
@@ -39,4 +41,6 @@
           <mesh filename="package://cats/meshes/STL/caster/caster_arm.stl" scale="0.001 0.001 0.001"/>
         </geometry>
+        <material name="gray">
+        </material>
       </visual>
       <collision>
@@ -64,4 +68,6 @@
           <mesh filename="package://cats/meshes/STL/caster/caster_wheel.stl" scale="0.001 0.001 0.001"/>
         </geometry>
+        <material name="gray">
+        </material>
       </visual>
       <collision>
@@ -82,4 +88,5 @@
       <mu1 value="0"/>
       <mu2 value="0"/>
+      <material>Gazebo/Gray</material>
     </gazebo>
     <gazebo reference="${prefix}_caster_arm_link">
@@ -87,4 +94,5 @@
       <mu1 value="0.05"/>
       <mu2 value="0.05"/>
+      <material>Gazebo/Gray</material>
     </gazebo>
     <gazebo reference="${prefix}_caster_wheel_link">
@@ -92,4 +100,5 @@
       <mu1 value="0.8"/>
       <mu2 value="0.8"/>
+      <material>Gazebo/Gray</material>
     </gazebo>
   </xacro:macro>

File: urdf/wheel/wheel.urdf.xacro (robot description, xacro)
@@ -19,4 +19,7 @@
           <mesh filename="package://cats/meshes/STL/wheel.stl" scale="0.001 0.001 0.001"/>
         </geometry>
+        <material name="black">
+          <color rgba="0.0 0.0 0.0 1.0"/>
+        </material>
       </visual>
       <collision>
@@ -39,4 +42,5 @@
       <mu1 value="0.8"/>
       <mu2 value="0.8"/>
+      <material>Gazebo/Black</material>
     </gazebo>
   </xacro:macro>
